Commit message: Adjust camera frame topology into a stereo pair (#37)
* Adjust camera frame topology into a stereo pair

* move task items (#38)

* Adjust work-tray height collider and place PCIe card on it

* Move all items in field of view, remove test block

* Define global_illumination in sensors system (#39)

* Adjust optical/sensor frame names and increase frame rate

* move second wrist camera to 120 degree rotation from first camera

---------

Signed-off-by: Yadunund <yadunund@intrinsic.ai>
Co-authored-by: Yadunund <yadunund@intrinsic.ai>

File: aic_assets/models/Basler Camera/basler_camera_macro.xacro (robot description, xacro)
@@ -1,8 +1,11 @@
 <?xml version="1.0"?>
 <robot xmlns:xacro="http://wiki.ros.org/xacro">
-  <xacro:macro name="basler_camera" params="name tf_prefix cam_lens_offset use_sim_cam">
+  <xacro:macro name="basler_camera" params="name tf_prefix use_sim_cam">
+    <xacro:property name="x_rot" value="1.5708"/>
+    <xacro:property name="y_rot" value="0.0"/>
+    <xacro:property name="z_rot" value="1.5708"/>
     <link name="${tf_prefix}basler_cam_link">
       <inertial>
-        <origin xyz="0 0 0" rpy="0 0 0"/>
+        <origin xyz="0 0 0" rpy="${x_rot} ${y_rot} ${z_rot}"/>
         <mass value="0.1"/>
         <inertia ixx="0.00002083" ixy="0" ixz="0"
@@ -11,5 +14,5 @@
       </inertial>
       <visual name="basler_cam_visual">
-        <origin xyz="0 0 -${cam_lens_offset}" rpy="0 0 0"/>
+        <origin xyz="0 0 0" rpy="${x_rot} ${y_rot} ${z_rot}"/>
         <geometry>
           <mesh filename="package://aic_assets/models/Basler Camera/basler_cam_visual.glb"/>
@@ -17,5 +20,5 @@
       </visual>
       <collision name="lens001_collider_cylinder">
-        <origin xyz="-0.000005 0.000001 ${0.013336 - cam_lens_offset}" rpy="0.0 0.0 0.0"/>
+        <origin xyz="0.013336 0 0" rpy="${x_rot} ${y_rot} ${z_rot}"/>
         <geometry>
           <cylinder radius="0.016429" length="0.040108"/>
@@ -23,11 +26,12 @@
       </collision>
       <collision name="basler_ace2_gige027_collider_box">
-        <origin xyz="-0.000001 -0.000017 ${-0.031178 - cam_lens_offset}" rpy="0.0 0.0 0.0"/>
+        <origin xyz="-0.031178 0 0" rpy="0 0 0"/>
         <geometry>
-          <box size="0.028998 0.028965 0.04919"/>
+          <box size="0.04919 0.029 0.029"/>
         </geometry>
       </collision>
+      <!-- the IO connector on the back of the camera -->
       <collision name="basler_ace2_gige011_collider_cylinder">
-        <origin xyz="-0.005773 -0.0081 ${-0.058082 - cam_lens_offset}" rpy="0.0 0.0 0.0"/>
+        <origin xyz="-0.058082 -0.005773 -0.0081" rpy="0 1.5708 0"/>
         <geometry>
           <cylinder radius="0.005145" length="0.008255"/>
@@ -35,4 +39,23 @@
       </collision>
     </link>
+    <link name="${tf_prefix}optical">
+      <!-- inertial property required for valid conversion to SDF,
+        so we set a tiny mass and M.O.I. here -->
+      <inertial>
+        <origin xyz="0 0 0" rpy="0 0 0"/>
+        <mass value="0.001"/>
+        <inertia ixx="0.000001" ixy="0" ixz="0"
+                 iyy="0.000001" iyz="0"
+                 izz="0.000001"/>
+      </inertial>
+    </link>
+    <joint name="${tf_prefix}attach_optical" type="fixed">
+      <origin xyz="0 0 0" rpy="-1.5708 0 -1.5708"/>
+      <parent link="${tf_prefix}basler_cam_link"/>
+      <child link="${tf_prefix}optical"/>
+    </joint>
+    <gazebo reference="${tf_prefix}attach_optical">
+      <preserveFixedJoint>true</preserveFixedJoint>
+    </gazebo>
     <link name="${tf_prefix}sensor_link">
       <!-- inertial property required for valid conversion to SDF,
@@ -46,10 +69,14 @@
       </inertial>
     </link>
-    <joint name="${tf_prefix}attach_sensor" type="fixed">
+    <!-- Currently the sensor_link is the same location as the
+         cam_link frame. However, we may adjust this in the future
+         if the lens focal point ends up being somewhat forward or
+         backward of the current estimate. -->
+    <joint name="${tf_prefix}attach_sensor_link" type="fixed">
       <origin xyz="0 0 0" rpy="0 0 0"/>
       <parent link="${tf_prefix}basler_cam_link"/>
       <child link="${tf_prefix}sensor_link"/>
     </joint>
-    <gazebo reference="${tf_prefix}attach_sensor">
+    <gazebo reference="${tf_prefix}attach_sensor_link">
       <preserveFixedJoint>true</preserveFixedJoint>
     </gazebo>
@@ -57,41 +84,22 @@
       <gazebo reference="${tf_prefix}sensor_link">
         <sensor name="${name}" type="camera">
-          <pose>0 0 0 1.57079632679 -1.57079632679 0</pose>
-          <update_rate>10.0</update_rate>
+          <pose>0 0 0 0 0 0</pose>
+          <update_rate>20.0</update_rate>
           <topic>/${name}/image</topic>
           <always_on>true</always_on>
-          <visualize>true</visualize>
           <frame_id>${tf_prefix}sensor_link</frame_id>
           <camera name="${name}">
             <camera_info_topic>/${name}/camera_info</camera_info_topic>
+            <optical_frame_id>${tf_prefix}optical</optical_frame_id>
             <image>
-              <width>2840</width>
-              <height>2840</height>
+              <width>1420</width>
+              <height>1420</height>
               <format>R8G8B8</format>
             </image>
-            <lens>
-              <intrinsics>
-                <fx>2920</fx>
-                <fy>2920</fy>
-                <cx>1420</cx>
-                <cy>1420</cy>
-              </intrinsics>
-            </lens>
+            <horizontal_fov>1.0</horizontal_fov>
             <clip>
-              <near>0.02</near>
+              <near>0.07</near>
               <far>300</far>
             </clip>
-            <distortion>
-              <k1>0</k1>
-              <k2>0</k2>
-              <k3>0</k3>
-              <p1>0</p1>
-              <p2>0</p2>
-            </distortion>
-            <noise>
-              <type>gaussian</type>
-              <mean>0.0</mean>
-              <stddev>0.007</stddev>
-            </noise>
           </camera>
         </sensor>

File: aic_assets/models/Camera Mount/cam_mount_macro.xacro (robot description, xacro)
@@ -2,4 +2,5 @@
 <robot xmlns:xacro="http://wiki.ros.org/xacro">
   <xacro:property name="tf_prefix" value="cam_mount/"/>
+  <xacro:property name="z_rot" value="-1.57079"/>
   <xacro:macro name="camera_mount" params="tf_prefix">
     <link name="${tf_prefix}cam_mount_link">
@@ -12,4 +13,5 @@
       </inertial>
       <visual name="cam_mount_visual">
+        <origin xyz="0.0 0.0 0.0215" rpy="0.0 0.0 ${z_rot}"/>
         <geometry>
           <mesh filename="package://aic_assets/models/Camera Mount/cam_mount_visual.glb"/>
@@ -17,5 +19,5 @@
       </visual>
       <collision name="cam_mount_collider_cylinder">
-        <origin xyz="0.0 0.0 0.0215" rpy="0.0 0.0 0.0"/>
+        <origin xyz="0.0 0.0 0.0215" rpy="0.0 0.0 ${z_rot}"/>
         <geometry>
           <cylinder radius="0.06" length="0.01"/>
@@ -23,5 +25,5 @@
       </collision>
       <collision name="cam_mount_collider_cylinder.001">
-        <origin xyz="0.0 0.0 0.012638" rpy="0.0 0.0 0.0"/>
+        <origin xyz="0.0 0.0 0.012638" rpy="0.0 0.0 ${z_rot}"/>
         <geometry>
           <cylinder radius="0.030383" length="0.025275"/>
@@ -29,5 +31,5 @@
       </collision>
       <collision name="cam_mount003_collider_box">
-        <origin xyz="0.068974 0.000189 0.02" rpy="0.0 0.0 0.0"/>
+        <origin xyz="0.068974 0.000189 0.02" rpy="0.0 0.0 ${z_rot}"/>
         <geometry>
           <box size="0.055675 0.027622 0.003"/>
@@ -35,5 +37,5 @@
       </collision>
       <collision name="cam_mount003_collider_box.001">
-        <origin xyz="0.096142 0.000189 0.021981" rpy="0.0 1.308997 0.0"/>
+        <origin xyz="0.096142 0.000189 0.021981" rpy="0.0 1.308997 ${z_rot}"/>
         <geometry>
           <box size="0.035256 0.027622 0.003"/>
@@ -41,5 +43,5 @@
       </collision>
       <collision name="cam_mount003_collider_box.002">
-        <origin xyz="-0.034323 -0.059827 0.02" rpy="0.0 0.0 -2.094395"/>
+        <origin xyz="-0.034323 -0.059827 0.02" rpy="0.0 0.0 ${z_rot - 2.094395}"/>
         <geometry>
           <box size="0.055675 0.027622 0.003"/>
@@ -47,5 +49,5 @@
       </collision>
       <collision name="cam_mount003_collider_box.003">
-        <origin xyz="-0.047908 -0.083356 0.021981" rpy="0.0 1.308997 -2.094395"/>
+        <origin xyz="-0.047908 -0.083356 0.021981" rpy="0.0 1.308997 ${z_rot - 2.094395}"/>
         <geometry>
           <box size="0.035256 0.027622 0.003"/>
@@ -53,5 +55,5 @@
       </collision>
       <collision name="cam_mount003_collider_box.004">
-        <origin xyz="-0.03465 0.059639 0.02" rpy="0.0 0.0 -4.18879"/>
+        <origin xyz="-0.03465 0.059639 0.02" rpy="0.0 0.0 ${z_rot - 4.18879}"/>
         <geometry>
           <box size="0.055675 0.027622 0.003"/>
@@ -59,5 +61,5 @@
       </collision>
       <collision name="cam_mount003_collider_box.005">
-        <origin xyz="-0.048235 0.083167 0.021981" rpy="0.0 1.308997 -4.18879"/>
+        <origin xyz="-0.048235 0.083167 0.021981" rpy="0.0 1.308997 ${z_rot - 4.18879}"/>
         <geometry>
           <box size="0.035256 0.027622 0.003"/>

File: aic_description/urdf/ur_gz.urdf.xacro (robot description, xacro)
@@ -33,6 +33,6 @@
   <xacro:arg name="wrist_camera_2_tf_prefix" default="wrist_camera_2/"/>
   <xacro:arg name="gripper_tf_prefix" default="gripper/"/>
-  <xacro:arg name="cam_lens_offset" default="0.035" />
-  <xacro:arg name="cam_mount_offset" default="0.09495" />
+  <xacro:arg name="cam_mount_radial_offset" default="0.1" />
+  <xacro:arg name="cam_mount_axial_offset" default="0.08" />
   <!-- If true, enable Gazebo camera in sim -->
   <xacro:arg name="use_sim_cam" default="${True}"/>
@@ -116,5 +116,4 @@
     name="wrist_camera_1"
     tf_prefix="$(arg wrist_camera_1_tf_prefix)"
-    cam_lens_offset="$(arg cam_lens_offset)"
     use_sim_cam="$(arg use_sim_cam)"
     >
@@ -123,5 +122,4 @@
     name="wrist_camera_2"
     tf_prefix="$(arg wrist_camera_2_tf_prefix)"
-    cam_lens_offset="$(arg cam_lens_offset)"
     use_sim_cam="$(arg use_sim_cam)"
     >
@@ -139,5 +137,5 @@
   </xacro:robotiq_hande>
   <joint name="attach_cam_mount" type="fixed">
-    <origin xyz="0 0 0" rpy="0 0 0"/>
+    <origin xyz="0 0 -.0265" rpy="0 0 0"/>
     <parent link="$(arg tf_prefix)tool0"/>
     <child link="$(arg cam_mount_tf_prefix)cam_mount_link"/>
@@ -148,14 +146,44 @@
     <child link="$(arg ati_tf_prefix)base_link"/>
   </joint>
+  <!-- Dummy link to simplify the chain of rotations -->
+  <link name="wrist_camera_1_intermediate_link">
+    <inertial>
+      <origin xyz="0 0 0" rpy="0 0 0"/>
+      <mass value="0.001"/>
+      <inertia ixx="0.000001" ixy="0" ixz="0"
+               iyy="0.000001" iyz="0"
+               izz="0.000001"/>
+    </inertial>
+  </link>
+  <joint name="wrist_camera_1_intermediate_joint" type="fixed">
+    <origin xyz="0 -$(arg cam_mount_radial_offset) $(arg cam_mount_axial_offset)"
+      rpy="${90.0*D2R} ${-90.0*D2R} ${0.0*D2R}"/>
+    <parent link="$(arg cam_mount_tf_prefix)cam_mount_link"/>
+    <child link="wrist_camera_1_intermediate_link"/>
+  </joint>
   <joint name="attach_wrist_camera_1" type="fixed">
-    <origin xyz="$(arg cam_mount_offset) 0 ${0.054483+$(arg cam_lens_offset)}"
-      rpy="0.261799 0 -1.5708"/>
+    <origin xyz="0 0 0" rpy="${0.0*D2R} ${15.0*D2R} ${0.0*D2R}"/>
+    <parent link="wrist_camera_1_intermediate_link"/>
+    <child link="$(arg wrist_camera_1_tf_prefix)basler_cam_link"/>
+  </joint>
+  <!-- Dummy link to simplify the chain of rotations -->
+  <link name="wrist_camera_2_intermediate_link">
+    <inertial>
+      <origin xyz="0 0 0" rpy="0 0 0"/>
+      <mass value="0.001"/>
+      <inertia ixx="0.000001" ixy="0" ixz="0"
+               iyy="0.000001" iyz="0"
+               izz="0.000001"/>
+    </inertial>
+  </link>
+  <joint name="wrist_camera_2_intermediate_joint" type="fixed">
+    <origin xyz="${-cos(30.0*D2R)*$(arg cam_mount_radial_offset)} ${sin(30.0*D2R)*$(arg cam_mount_radial_offset)} $(arg cam_mount_axial_offset)"
+      rpy="${90.0*D2R} ${-90.0*D2R} ${-120.0*D2R}"/>
     <parent link="$(arg cam_mount_tf_prefix)cam_mount_link"/>
-    <child link="$(arg wrist_camera_1_tf_prefix)basler_cam_link"/>
+    <child link="wrist_camera_2_intermediate_link"/>
   </joint>
   <joint name="attach_wrist_camera_2" type="fixed">
-    <origin xyz="-${$(arg cam_mount_offset) * sin(30.0*D2R)} -${$(arg cam_mount_offset) * cos(30.0*D2R)} ${0.054483+$(arg cam_lens_offset)}"
-      rpy="0.261799 0 2.61799"/>
-    <parent link="$(arg cam_mount_tf_prefix)cam_mount_link"/>
+    <origin xyz="0 0 0" rpy="${0.0*D2R} ${15.0*D2R} ${0.0*D2R}"/>
+    <parent link="wrist_camera_2_intermediate_link"/>
     <child link="$(arg wrist_camera_2_tf_prefix)basler_cam_link"/>
   </joint>
